File: Schematic.sch (EAGLE design)
At the start: 24 parts

Commit message: board with routing
Parts:
- removed DELAYTIME1: 10 LIN, piher:PC16S
- removed EFFECT1, REVERB1, REVERBTIME1: 10K LIN, piher:PC16S
- removed FEEDBACK1, FILTER1, FREQ1, INPUT1, INPUTTHRU1, INPUTTODELAY1, MOD1, OUTPUT1, SIRENVOL1, SPEED1: 10K LOG, piher:PC16S
- removed U$3, U$4: TEENSY_3.5/3.6, Teensy356:TEENSY_3.5/3.6
- removed USB_INPUT: PN61729-S, con-berg:PN61729-S
- added D1: 5KPXX, diode:5KPXX
- added DELAYTIME, EFFECT, FEEDBACK, FILTER, FREQ, INPUT, INPUT-THRU, INPUT-TO-DELAY, MOD, OUTPUT, REVERB-AMOUNT, REVERB-TIME, SIRENVOL, SPEED: RK09L1140A66, SamacSys_Parts:RK09L1140A66
- added FILTER_PASS, HOLD, WAVEFORM: (no value), SparkFun-Switches:SWITCH-SPDT-PTH-11.6X4.0MM-LOCK
- added FIRE: CHERRY-MX-LED, cherrymx:CHERRY-MX-LED
- added MICLINE_SWITCH: OS102011MA1QN1, OS102011MA1QN1:OS102011MA1QN1
- added OLED: (no value), pinhead:PINHD-1X4
- added R1, R2: (no value), resistor:R-US_0207/10
- added SOUND: CHERRY-MX, cherrymx:CHERRY-MX
- added TEST_3V, TEST_5V, TEST_GND: (no value), pinhead:PINHD-1X1
- added USB: XM7D-0512, SamacSys_Parts:XM7D-0512
- POWER_SWITCH: value 2P2T -> OS102011MA1QN1; device switch:2P2T -> OS102011MA1QN1:OS102011MA1QN1
- renumbered U$1 to TEENSY
Connections:
- removed net N$7: U$4.GND
- removed net PIN18: TEENSY.18/A4/SDA, U$4.18/A4/SDA, U$5.18
- removed net PIN19: TEENSY.19/A5/SCL, U$4.19/A5/SCL, U$5.19
- new net BUTTON_FIRE: FIRE.LED+, FIRE.SW2, TEENSY.25
- new net BUTTON_HOLD: HOLD.S, TEENSY.24
- new net BUTTON_SOUND: SOUND.PIN-2, TEENSY.26
- new net LED_HOLD: D1.A, TEENSY.3/CANTX
- new net PIN27: TEENSY.27, WAVEFORM.S
- new net PIN30: TEENSY.30, WAVEFORM.O
- new net PIN4: FILTER_PASS.O, TEENSY.4/CANRX
- new net PIN5: FILTER_PASS.S, TEENSY.5
- new net PIN8: MICLINE_SWITCH.3, TEENSY.8
- new net SCL: OLED.2, R1.1, TEENSY.19/A5/SCL, U$5.19
- new net SDA: OLED.1, R2.1, TEENSY.18/A4/SDA, U$5.18
- new net TEST_5V: TEENSY.U5V, TEST_5V.1, U$2.5V
- net 3V: no longer U$4.3V3_LO, U$5.3V
- net GND: now also D1.C, DELAYTIME.3, EFFECT.3, FEEDBACK.3, FILTER.3, FIRE.LED-, FREQ.3, INPUT-THRU.3, INPUT-TO-DELAY.3, INPUT.3, MOD.3, OLED.4, OUTPUT.3, REVERB-AMOUNT.3, REVERB-TIME.3, SIRENVOL.3, SPEED.3, TEST_GND.1; no longer DELAYTIME1.1E, EFFECT1.1E, FEEDBACK1.1E, FILTER1.1E, FREQ1.1E, INPUT1.1E, INPUTTHRU1.1E, INPUTTODELAY1.1E, MOD1.1E, OUTPUT1.1E, REVERB1.1E, REVERBTIME1.1E, SIRENVOL1.1E, SPEED1.1E
- net KNOB_DELAY: now also DELAYTIME.2; no longer DELAYTIME1.1S, U$3.21/A7
- net KNOB_EFFECT: now also EFFECT.2; no longer EFFECT1.1S, U$3.37/A18
- net KNOB_FEEDBACK: now also FEEDBACK.2; no longer FEEDBACK1.1S, U$3.33/A14
- net KNOB_FILTER: now also FILTER.2; no longer FILTER1.1S, U$3.34/A15
- net KNOB_FREQ: now also FREQ.2; no longer FREQ1.1S, U$3.17/A3
- net KNOB_INPUT: now also INPUT.2; no longer INPUT1.1S, U$3.31/A12
- net KNOB_INPUTTHRU: now also INPUT-THRU.2; no longer INPUTTHRU1.1S, U$3.36/A17
- net KNOB_INPUTTODELAY: now also INPUT-TO-DELAY.2; no longer INPUTTODELAY1.1S, U$3.35/A16
- net KNOB_MOD: now also MOD.2; no longer MOD1.1S, U$3.16/A2
- net KNOB_OUTPUT: now also OUTPUT.2; no longer OUTPUT1.1S, U$3.32/A13
- net KNOB_REVERBTIME: now also REVERB-TIME.2; no longer REVERBTIME1.1S, U$3.20/A6
- net KNOB_REVERBVOLUME: now also REVERB-AMOUNT.2; no longer REVERB1.1S, U$3.A10
- net KNOB_SIRENVOL: now also SIRENVOL.2; no longer SIRENVOL1.1S, U$3.39/A20
- net KNOB_SPEED: now also SPEED.2; no longer SPEED1.1S, U$3.38/A19
- net N$1: now also USB.1; no longer USB_INPUT.1
- net N$16: now also POWER_SWITCH.1; no longer POWER_SWITCH.3.2
- net N$17: now also POWER_SWITCH.2; no longer POWER_SWITCH.3.1
- net N$2: now also USB.5; no longer USB_INPUT.4
- net N$3: now also USB.2; no longer USB_INPUT.2
- net N$4: now also USB.3; no longer USB_INPUT.3
- net PIN10: no longer U$4.10/CS
- net PIN11: no longer U$4.11/MOSI
- net PIN12: no longer U$4.12/MISO
- net PIN13: no longer U$4.13/SCK
- net PIN14: no longer U$4.14/A0
- net PIN15: no longer U$4.15/A1
- net PIN22: no longer U$4.22/A8
- net PIN23: no longer U$4.23/A9
- net PIN6: no longer U$4.6
- net PIN7: no longer U$4.7
- net PIN9: no longer U$4.9/CS
- net VCC: now also DELAYTIME.1, EFFECT.1, FEEDBACK.1, FILTER.1, FILTER_PASS.P, FIRE.SW1, FREQ.1, HOLD.P, INPUT-THRU.1, INPUT-TO-DELAY.1, INPUT.1, MICLINE_SWITCH.2, MOD.1, OLED.3, OUTPUT.1, R1.2, R2.2, REVERB-AMOUNT.1, REVERB-TIME.1, SIRENVOL.1, SOUND.PIN-1, SPEED.1, TEENSY.3V3, TEST_3V.1, U$5.3V, WAVEFORM.P; no longer DELAYTIME1.1A, EFFECT1.1A, FEEDBACK1.1A, FILTER1.1A, FREQ1.1A, INPUT1.1A, INPUTTHRU1.1A, INPUTTODELAY1.1A, MOD1.1A, OUTPUT1.1A, REVERB1.1A, REVERBTIME1.1A, SIRENVOL1.1A, SPEED1.1A, TEENSY.U5V, U$2.5V
